File: Draw_Eagle/NavCom/NavCom_Board_3.brd (EAGLE design)
At the start: 172.7 x 50.8 mm, 43 parts

Commit message: This is tag #4 taken from former SVN repository.
Parts:
- removed U$24, U$25, U$26, U$28: KONDENZATOR, RadioStack_v2:KONDENZATOR
- removed U$37: REZISTOR, RadioStack_v2:REZISTOR
- added 33PF: 33pF, RadioStack_v2:KONDENZATOR
- U$19, U$20, U$21, U$22, U$8: value KONDENZATOR -> REZISTOR; device RadioStack_v2:KONDENZATOR -> RadioStack_v2:REZISTOR
- U$23: value KONDENZATOR -> 3.9k; device RadioStack_v2:KONDENZATOR -> RadioStack_v2:REZISTOR
- U$27, U$34, U$40, U$41: value REZISTOR -> 470M
- moved U$22 111.9 mm to (38.1, 25.4), turned to 180 degrees
- moved U$21 95.4 mm to (55.9, 11.4), turned to 90 degrees
- moved U$20 92.5 mm to (58.4, 11.4), turned to 90 degrees
- moved U$19 89.6 mm to (61.0, 11.4), turned to 90 degrees
- moved U$8 86.8 mm to (63.5, 11.4), turned to 90 degrees
- moved U$23 51.8 mm to (76.2, 10.2)
- moved U$2 35.8 mm to (20.3, 38.1)
- moved U$3 21.6 mm to (45.7, 44.5)
- moved U$40 12.0 mm to (16.5, 26.7), flipped to the bottom, turned to 180 degrees
- moved U$11 6.48 mm to (74.9, 31.8)
- moved U$1 6.48 mm to (104.1, 15.2)
- moved U$41 5.08 mm to (11.4, 17.8), flipped to the bottom
- flipped U$27 to the bottom
- flipped U$34 to the bottom
- flipped U$35 to the bottom, turned to 180 degrees
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- renumbered CONNECTOR to CONNECTOR_LEFT
Connections:
- removed net N$29 (its old number): U$28.P$2, U$3.P$4, U$35.P$1
- removed net N$44: U$10.P$2, U$12.P$2, U$13.P$1, U$14.P$1, U$15.P$1, U$16.P$1, U$17.P$2, U$18.P$1, U$3.P$2, U$3.P$6, U$4.P$2, U$4.P$6, U$5.P$2, U$5.P$6, U$6.P$2, U$6.P$6, U$7.P$2, U$9.P$2
- new net N$31: CONNECTOR_LEFT.8, U$1.GP0.6, U$19.P$2
- new net N$41: 33PF.P$2, U$1.CLK, U$23.P$2
- new net N$45: U$1.~INT, U$2.4
- new net N$46: CONNECTOR_LEFT.7, U$1.GP0.5, U$20.P$2
- new net N$47: U$1.GP1.7, U$2.5
- new net N$48: CONNECTOR_LEFT.6, U$1.GP0.4, U$21.P$2
- new net N$49: U$3.P$5, U$38.P$1
- net N$11: now also U$1.GP1.4, U$22.P$1; no longer CONNECTOR_LEFT.3, U$14.P$2, U$37.P$2
- net N$14: now also U$6.P$4; no longer U$23.P$2, U$3.P$5
- net N$15: now also U$4.P$4; no longer U$19.P$2, U$4.P$5
- net N$16: now also CONNECTOR_LEFT.9, U$1.GP0.7, U$8.P$2; no longer U$19.P$1, U$20.P$1, U$21.P$1, U$22.P$1, U$23.P$1, U$24.P$1, U$25.P$1, U$26.P$1, U$27.P$2, U$28.P$1, U$3.P$3, U$34.P$1, U$4.P$3, U$40.P$1, U$41.P$1, U$5.P$3, U$6.P$3, U$8.P$1
- net N$17: now also U$5.P$5; no longer U$20.P$2, U$5.P$4
- net N$18: now also U$1.GP1.5; no longer U$21.P$2
- net N$19: now also U$4.P$5; no longer U$22.P$2, U$4.P$4
- net N$20: now also U$3.P$4, U$35.P$1; no longer U$24.P$2, U$38.P$1
- net N$21: now also CONNECTOR_LEFT.3, U$14.P$2, U$22.P$2; no longer U$25.P$2, U$37.P$1
- net N$23: now also U$6.P$5; no longer U$26.P$2
- net N$24: now also U$1.GP0.2; no longer U$1.GP0.4
- net N$26: now also U$1.GP1.2; no longer U$1.GP0.5
- net N$32: now also U$1.GP0.3; no longer U$1.GP0.7
- net N$33: now also U$1.GP1.3; no longer U$1.GP0.6
- net N$34: now also U$1.GP1.0; no longer U$1.GP0.3
- net N$35: now also U$1.GP0.0; no longer U$1.GP0.2
- net N$36: now also U$1.GP1.1; no longer U$1.GP0.0
- net N$42: now also U$2.10
- net N$43: now also U$2.9
- net N$5: now also U$5.P$4; no longer U$5.P$5, U$8.P$2
- net N$7: now also 33PF.P$1, CONNECTOR2.4, U$1.VSS1, U$1.VSS2, U$1.VSS3, U$2.6, U$27.P$2, U$3.P$3, U$34.P$1, U$4.P$3, U$40.P$1, U$41.P$1, U$5.P$3, U$6.P$3
- net N$8: now also CONNECTOR2.5, U$1.GP1.6, U$1.VDD, U$10.P$2, U$12.P$2, U$13.P$1, U$14.P$1, U$15.P$1, U$16.P$1, U$17.P$2, U$18.P$1, U$19.P$1, U$2.7, U$20.P$1, U$21.P$1, U$23.P$1, U$3.P$2, U$3.P$6, U$4.P$2, U$4.P$6, U$5.P$2, U$5.P$6, U$6.P$2, U$6.P$6, U$7.P$2, U$8.P$1, U$9.P$2
Routing:
- net N$8: track 5.08 -> 492.9 mm, vias 0 -> 2
- net N$7: track 5.08 -> 320.8 mm, vias 0 -> 2
- net N$44: track 235.1 -> 0.00 mm
- net N$42: track 73.2 -> 190.8 mm
- net N$43: track 57.2 -> 169.5 mm, vias 1 -> 3
- net N$18: track 5.08 -> 116.3 mm, vias 0 -> 2
- net N$45: track 0.00 -> 108.7 mm
- net N$31: track 0.00 -> 104.7 mm
- net N$46: track 0.00 -> 101.1 mm
- net N$48: track 0.00 -> 97.5 mm
- net N$47: track 0.00 -> 77.3 mm
- net N$11: track 16.1 -> 78.5 mm, vias 0 -> 1
- net N$23: track 5.08 -> 63.4 mm
- net N$16: track 127.3 -> 95.0 mm
- net N$33: track 58.6 -> 87.9 mm, vias 0 -> 2
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Other:
- board text added: "INT"
- board text added: "LATCH RESET"
- board text added: "NC"
- board text removed: "NOT CONNECTED"
