File: Draw_Eagle/NavCom/NavCom_Board_3.sch (EAGLE design)
At the start: 43 parts

Commit message: This is tag #4 taken from former SVN repository.
Parts:
- removed CONNECTOR: LISTA_2X5, RadioStack_v2:LISTA_2X5
- removed U$24, U$25, U$26, U$28: KONDENZATOR, RadioStack_v2:KONDENZATOR
- removed U$37: REZISTOR, RadioStack_v2:REZISTOR
- added 33PF: 33pF, RadioStack_v2:KONDENZATOR
- added CONNECTOR_LEFT: LISTA_2X5, RadioStack_v2:LISTA_2X5
- U$19, U$20, U$21, U$22, U$8: value KONDENZATOR -> REZISTOR; device RadioStack_v2:KONDENZATOR -> RadioStack_v2:REZISTOR
- U$23: value KONDENZATOR -> 3.9k; device RadioStack_v2:KONDENZATOR -> RadioStack_v2:REZISTOR
- U$27, U$34, U$40, U$41: value REZISTOR -> 470M
Connections:
- removed net N$29 (its old number): U$28.P$2, U$3.A, U$35.P$1
- removed net N$44: U$10.P$2, U$12.P$2, U$13.P$1, U$14.P$1, U$15.P$1, U$16.P$1, U$17.P$2, U$18.P$1, U$3.VDD, U$3.X4/X1, U$4.VDD, U$4.X4/X1, U$5.VDD, U$5.X4/X1, U$6.VDD, U$6.X4/X1, U$7.P$2, U$9.P$2
- new net N$31: CONNECTOR_LEFT.8, U$1.GP0.6, U$19.P$2
- new net N$41: 33PF.P$2, U$1.CLK, U$23.P$2
- new net N$45: U$1.~INT, U$2.4
- new net N$46: CONNECTOR_LEFT.7, U$1.GP0.5, U$20.P$2
- new net N$47: U$1.GP1.7, U$2.5
- new net N$48: CONNECTOR_LEFT.6, U$1.GP0.4, U$21.P$2
- new net N$49: U$3.B, U$38.P$1
- net N$10: now also CONNECTOR_LEFT.2; no longer CONNECTOR.2
- net N$11: now also U$1.GP1.4, U$22.P$1; no longer CONNECTOR.3, U$14.P$2, U$37.P$2
- net N$12: now also CONNECTOR_LEFT.4; no longer CONNECTOR.4
- net N$13: now also CONNECTOR_LEFT.5; no longer CONNECTOR.5
- net N$14: now also U$6.A; no longer U$23.P$2, U$3.B
- net N$15: now also U$4.A; no longer U$19.P$2, U$4.B
- net N$16: now also CONNECTOR_LEFT.9, U$1.GP0.7, U$8.P$2; no longer U$19.P$1, U$20.P$1, U$21.P$1, U$22.P$1, U$23.P$1, U$24.P$1, U$25.P$1, U$26.P$1, U$27.P$2, U$28.P$1, U$3.VSS, U$34.P$1, U$4.VSS, U$40.P$1, U$41.P$1, U$5.VSS, U$6.VSS, U$8.P$1
- net N$17: now also U$5.B; no longer U$20.P$2, U$5.A
- net N$18: now also U$1.GP1.5; no longer U$21.P$2
- net N$19: now also U$4.B; no longer U$22.P$2, U$4.A
- net N$20: now also U$3.A, U$35.P$1; no longer U$24.P$2, U$38.P$1
- net N$21: now also CONNECTOR_LEFT.3, U$14.P$2, U$22.P$2; no longer U$25.P$2, U$37.P$1
- net N$23: now also U$6.B; no longer U$26.P$2
- net N$24: now also U$1.GP0.2; no longer U$1.GP0.4
- net N$26: now also U$1.GP1.2; no longer U$1.GP0.5
- net N$32: now also U$1.GP0.3; no longer U$1.GP0.7
- net N$33: now also U$1.GP1.3; no longer U$1.GP0.6
- net N$34: now also U$1.GP1.0; no longer U$1.GP0.3
- net N$35: now also U$1.GP0.0; no longer U$1.GP0.2
- net N$36: now also U$1.GP1.1; no longer U$1.GP0.0
- net N$42: now also U$2.10
- net N$43: now also U$2.9
- net N$5: now also U$5.A; no longer U$5.B, U$8.P$2
- net N$7: now also 33PF.P$1, CONNECTOR2.4, U$1.VSS1, U$1.VSS2, U$1.VSS3, U$2.6, U$27.P$2, U$3.VSS, U$34.P$1, U$4.VSS, U$40.P$1, U$41.P$1, U$5.VSS, U$6.VSS
- net N$8: now also CONNECTOR2.5, U$1.GP1.6, U$1.VDD, U$10.P$2, U$12.P$2, U$13.P$1, U$14.P$1, U$15.P$1, U$16.P$1, U$17.P$2, U$18.P$1, U$19.P$1, U$2.7, U$20.P$1, U$21.P$1, U$23.P$1, U$3.VDD, U$3.X4/X1, U$4.VDD, U$4.X4/X1, U$5.VDD, U$5.X4/X1, U$6.VDD, U$6.X4/X1, U$7.P$2, U$8.P$1, U$9.P$2
- net N$9: now also CONNECTOR_LEFT.1; no longer CONNECTOR.1
Other:
- moved on the sheet: U$2
